File: hw/sch_pcb/TFASPDIMU01.kicad_pcb (KiCad board)
At the start: 2 copper layers, 36 x 14 mm, 26 parts, among them J1 SM07B-GHS-TB, U1 SDP3x, U2 ICM-20948, U4 MIC5504-3.3YM5-TR, U5 MIC5504-1.8YM5-TR, U6 TXS0108EPW

Commit message: Edit PCB for 3D model
Other:
- net class Default removed
- net class MLAB_default removed
- net class MLAB_power removed
