File: hw/sch_pcb/TFASPDIMU01.kicad_pcb (KiCad board)
At the start: 2 copper layers, 36 x 14 mm, 26 parts, among them J1 SM07B-GHS-TB, U1 SDP3x, U2 ICM-20948, U4 MIC5504-3.3YM5-TR, U5 MIC5504-1.8YM5-TR, U6 TXS0108EPW

Commit message: Update the project to KiCAD7.
Connections:
- U1 pad 4: (no net) -> unconnected-(U1-IRQn-Pad4)
- U2 pad 1: (no net) -> unconnected-(U2-NC-Pad1)
- U2 pad 14: (no net) -> unconnected-(U2-NC-Pad14)
- U2 pad 15: (no net) -> unconnected-(U2-NC-Pad15)
- U2 pad 16: (no net) -> unconnected-(U2-NC-Pad16)
- U2 pad 17: (no net) -> unconnected-(U2-NC-Pad17)
- U2 pad 19: (no net) -> unconnected-(U2-RESV-Pad19)
- U2 pad 2: (no net) -> unconnected-(U2-NC-Pad2)
- U2 pad 3: (no net) -> unconnected-(U2-NC-Pad3)
- U2 pad 4: (no net) -> unconnected-(U2-NC-Pad4)
- U2 pad 5: (no net) -> unconnected-(U2-NC-Pad5)
- U2 pad 6: (no net) -> unconnected-(U2-NC-Pad6)
- U4 pad 4: (no net) -> unconnected-(U4-NC-Pad4)
- U5 pad 4: (no net) -> unconnected-(U5-NC-Pad4)
- U6 pad 12: (no net) -> unconnected-(U6-B8-Pad12)
- U6 pad 9: (no net) -> unconnected-(U6-A8-Pad9)
