File: hw/sch_pcb/TFASPDIMU01.kicad_sch (KiCad schematic)
At the start: 26 parts, among them J1 SM07B-GHS-TB, U1 SDP3x, U2 ICM-20948, U4 MIC5504-3.3YM5-TR, U5 MIC5504-1.8YM5-TR, U6 TXS0108EPW

Commit message: Update title block.
Other:
- company: Mlab www.mlab.cz -> ThunderFly s.r.o.
- title: NAME -> TFASPDIMU01A
Changed lines of the file:
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@@
   (paper "A4")
   (title_block
-    (title "NAME")
-    (date "%F")
-    (rev "REV")
-    (company "Mlab www.mlab.cz")
-    (comment 1 "VERSION")
-    (comment 2 "Short description \\nTwo lines are maximum")
-    (comment 3 "nickname <email@example.com>")
-    (comment 4 "BSD")
+    (title "TFASPDIMU01A")
+    (date "2021-04-05")
+    (rev "A")
+    (company "ThunderFly s.r.o.")
+    (comment 1 "Differential pressure and  IMU \\n for airspeed sensing of UAVs")
+    (comment 3 "jacho <info@thunderfly.cz>")
+    (comment 4 "GPL 3.0")
   )
   (junction (at 20.32 130.81) (diameter 1.016) (color 0 0 0 0))
